Commit message: fix(urdf): correct center of mass to prevent flipping

File: src/buggy_description/urdf/buggy_urdf.xacro (robot description, xacro)
@@ -2,266 +2,266 @@
 <robot name="srm_aquila_buggy" xmlns:xacro="http://www.ros.org/wiki/xacro">
   <!--
-    SRM Autonomous Electric Campus Buggy
+    SRM Autonomous Electric Campus Buggy  v3.0
     Based on: Aquila EV TE-A6+2 (Tri Electric Pvt Ltd, Tamil Nadu)
-    Real Dimensions: 4120mm L x 1200mm W x 1900mm H
-    Wheel: 205/50-10 (10 inch alloy rim, ~0.254m radius)
-    Max Speed: 30 kmph | Turning Radius: <5m
-    Chassis: Ladder type tubular steel
+    FIXES in v3.0:
+      - Pillars: z origin fixed so they sit between chassis and roof
+      - Roof: height corrected so pillars connect
+      - LiDAR: now bolted flush ON TOP of roof (not floating)
+      - Camera: repositioned to front face of chassis at correct height
+      - Steering: rebuilt as proper column + wheel assembly
+      - Mirrors: rebuilt from scratch — properly attached to pillar base
+      - Seats: Gazebo material overrides added so brown shows correctly
+      - All sensor positions verified relative to base_link
   -->
-  <!-- ═══════════════════════════════════════════
-       PROPERTIES  (all in metres)
-       ═══════════════════════════════════════════ -->
-  <xacro:property name="chassis_length"  value="4.12"/>
-  <xacro:property name="chassis_width"   value="1.20"/>
-  <xacro:property name="chassis_height"  value="0.25"/>
-  <!-- chassis_z = wheel_radius + (chassis_height/2) + 0.04 = 0.26 + 0.125 + 0.04 = 0.425
-       This places the tire bottoms at z=0 (ground plane) so base_footprint is correct. -->
-  <xacro:property name="chassis_z"       value="0.425"/>   <!-- ride height -->
-  <!-- Roof canopy -->
-  <xacro:property name="roof_length"     value="3.20"/>
-  <xacro:property name="roof_width"      value="1.20"/>
-  <xacro:property name="roof_thickness"  value="0.06"/>
-  <xacro:property name="roof_height"     value="1.90"/>   <!-- total buggy height from ground -->
-  <!-- Pillars (A-pillar front, B-pillar rear) -->
-  <xacro:property name="pillar_r"        value="0.04"/>
-  <xacro:property name="pillar_h"        value="1.30"/>
-  <!-- Windshield -->
-  <xacro:property name="ws_length"       value="1.30"/>
-  <xacro:property name="ws_height"       value="0.60"/>
-  <xacro:property name="ws_thickness"    value="0.02"/>
-  <!-- Wheel geometry: 205/50-10 tyre on 10in rim -->
-  <!-- 10in rim = 0.254m diameter = 0.127m radius -->
-  <!-- 205mm section, 50% aspect → sidewall = 0.1025m -->
-  <!-- total radius = 0.127 + 0.1025 = ~0.254m, use 0.26 for clearance -->
-  <xacro:property name="wheel_radius"    value="0.26"/>
-  <xacro:property name="wheel_width"     value="0.205"/>
-  <!-- Wheelbase & track -->
-  <xacro:property name="wheelbase"       value="2.60"/>   <!-- front-to-rear axle -->
-  <xacro:property name="track_width"     value="1.10"/>   <!-- centre-to-centre -->
-  <!-- Seat dimensions -->
-  <xacro:property name="seat_l"          value="0.45"/>
-  <xacro:property name="seat_w"          value="0.48"/>
-  <xacro:property name="seat_h"          value="0.12"/>
-  <xacro:property name="backrest_h"      value="0.50"/>
-  <xacro:property name="backrest_t"      value="0.08"/>
-  <!-- ═══════════════════════════════════════════
+  <!-- ═══════════════════════════════
+       PROPERTIES
+  ═══════════════════════════════ -->
+  <xacro:property name="cl"   value="4.12"/>   <!-- chassis length -->
+  <xacro:property name="cw"   value="1.20"/>   <!-- chassis width  -->
+  <xacro:property name="ch"   value="0.25"/>   <!-- chassis height -->
+  <xacro:property name="cz"   value="0.425"/>  <!-- ride height (base_link above ground) -->
+  <xacro:property name="wr"   value="0.26"/>   <!-- wheel radius -->
+  <xacro:property name="ww"   value="0.205"/>  <!-- wheel width  -->
+  <!-- Pillar geometry:
+       Bottom of pillar = chassis top = cz + ch/2 above ground = 0.425+0.125=0.55m
+       Roof bottom      = 1.90 - cz  = 1.475m above base_link
+       Pillar length    = 1.475 - 0.125 = 1.35m
+       Pillar centre z  = 0.125 + 1.35/2 = 0.80m above base_link -->
+  <xacro:property name="pillar_h"  value="1.35"/>
+  <xacro:property name="pillar_cz" value="0.80"/>
+  <xacro:property name="pillar_r"  value="0.04"/>
+  <!-- Roof: sits at 1.475m above base_link (1.9m total height - 0.425 ride height) -->
+  <xacro:property name="roof_z"  value="1.475"/>
+  <xacro:property name="roof_t"  value="0.06"/>
+  <!-- Seat geometry -->
+  <xacro:property name="sl"  value="0.45"/>
+  <xacro:property name="sw"  value="0.48"/>
+  <xacro:property name="sh"  value="0.12"/>
+  <xacro:property name="brh" value="0.50"/>
+  <xacro:property name="brt" value="0.08"/>
+  <!-- ═══════════════════════════════
        MATERIALS
-       ═══════════════════════════════════════════ -->
-  <material name="arctic_white">  <color rgba="0.96 0.96 0.96 1.0"/></material>
-  <material name="beige_seat">    <color rgba="0.82 0.76 0.60 1.0"/></material>
-  <material name="black_tyre">    <color rgba="0.10 0.10 0.10 1.0"/></material>
-  <material name="silver_rim">    <color rgba="0.75 0.75 0.78 1.0"/></material>
-  <material name="dark_grey">     <color rgba="0.22 0.22 0.22 1.0"/></material>
-  <material name="clear_acrylic"> <color rgba="0.80 0.90 1.00 0.35"/></material>
-  <material name="frp_roof">      <color rgba="0.94 0.94 0.94 1.0"/></material>
-  <material name="chassis_steel"> <color rgba="0.30 0.30 0.30 1.0"/></material>
-  <material name="dashboard_blk"> <color rgba="0.15 0.15 0.15 1.0"/></material>
-  <!-- ═══════════════════════════════════════════
-       BASE FOOTPRINT  (ground contact reference)
-       ═══════════════════════════════════════════ -->
+  ═══════════════════════════════ -->
+  <material name="white">        <color rgba="0.96 0.96 0.96 1.0"/></material>
+  <material name="srm_blue">     <color rgba="0.05 0.25 0.65 1.0"/></material>
+  <material name="dark_grey">    <color rgba="0.18 0.18 0.18 1.0"/></material>
+  <material name="mid_grey">     <color rgba="0.45 0.45 0.45 1.0"/></material>
+  <material name="chassis_blk">  <color rgba="0.12 0.12 0.12 1.0"/></material>
+  <material name="brown">        <color rgba="0.55 0.28 0.08 1.0"/></material>
+  <material name="black_tyre">   <color rgba="0.08 0.08 0.08 1.0"/></material>
+  <material name="silver">       <color rgba="0.78 0.78 0.82 1.0"/></material>
+  <material name="clear">        <color rgba="0.80 0.90 1.00 0.25"/></material>
+  <material name="lidar_silver"> <color rgba="0.82 0.82 0.85 1.0"/></material>
+  <material name="lidar_blue">   <color rgba="0.10 0.50 0.90 1.0"/></material>
+  <material name="rs_grey">      <color rgba="0.55 0.58 0.62 1.0"/></material>
+  <material name="rs_black">     <color rgba="0.10 0.10 0.12 1.0"/></material>
+  <material name="lens_green">   <color rgba="0.20 0.65 0.35 1.0"/></material>
+  <material name="pcb_green">    <color rgba="0.10 0.35 0.15 1.0"/></material>
+  <material name="gps_white">    <color rgba="0.90 0.90 0.90 1.0"/></material>
+  <material name="us_blue">      <color rgba="0.15 0.30 0.70 1.0"/></material>
+  <material name="hl_white">     <color rgba="0.95 0.95 0.80 1.0"/></material>
+  <material name="tl_red">       <color rgba="0.90 0.10 0.10 1.0"/></material>
+  <!-- Inertial helper macro for visual-only links -->
+  <xacro:macro name="tiny_inertial">
+    <inertial>
+      <mass value="0.01"/>
+      <inertia ixx="0.0001" ixy="0" ixz="0" iyy="0.0001" iyz="0" izz="0.0001"/>
+    </inertial>
+  </xacro:macro>
+  <!-- ═══════════════════════════════
+       BASE FOOTPRINT
+  ═══════════════════════════════ -->
   <link name="base_footprint"/>
   <joint name="base_joint" type="fixed">
-    <parent link="base_footprint"/>
-    <child  link="base_link"/>
-    <origin xyz="0 0 ${chassis_z}" rpy="0 0 0"/>
-  </joint>
-  <!-- ═══════════════════════════════════════════
-       MAIN CHASSIS
-       ═══════════════════════════════════════════ -->
+    <parent link="base_footprint"/><child link="base_link"/>
+    <origin xyz="0 0 ${cz}" rpy="0 0 0"/>
+  </joint>
+  <!-- ═══════════════════════════════
+       CHASSIS
+  ═══════════════════════════════ -->
   <link name="base_link">
     <visual>
-      <geometry><box size="${chassis_length} ${chassis_width} ${chassis_height}"/></geometry>
-      <material name="arctic_white"/>
+      <geometry><box size="${cl} ${cw} ${ch}"/></geometry>
+      <material name="white"/>
     </visual>
     <collision>
-      <geometry><box size="${chassis_length} ${chassis_width} ${chassis_height}"/></geometry>
+      <geometry><box size="${cl} ${cw} ${ch}"/></geometry>
     </collision>
     <inertial>
       <mass value="280.0"/>
       <origin xyz="0 0 0" rpy="0 0 0"/>
-      <inertia ixx="80"  ixy="0" ixz="0"
-               iyy="400" iyz="0"
-               izz="450"/>
+      <inertia ixx="80" ixy="0" ixz="0" iyy="400" iyz="0" izz="450"/>
     </inertial>
   </link>
-  <!-- ───────── UNDER-CHASSIS FRAME RAILS (visual only) ───────── -->
-  <joint name="frame_left_joint" type="fixed">
-    <parent link="base_link"/><child link="frame_left"/>
-    <origin xyz="0 ${chassis_width/2 - 0.08} ${-chassis_height/2 - 0.04}" rpy="0 0 0"/>
-  </joint>
-  <link name="frame_left">
-    <visual>
-      <geometry><box size="${chassis_length} 0.06 0.06"/></geometry>
-      <material name="chassis_steel"/>
-    </visual>
-    <inertial><mass value="0.01"/><inertia ixx="0.001" ixy="0" ixz="0" iyy="0.001" iyz="0" izz="0.001"/></inertial>
-  </link>
-  <joint name="frame_right_joint" type="fixed">
-    <parent link="base_link"/><child link="frame_right"/>
-    <origin xyz="0 ${-(chassis_width/2 - 0.08)} ${-chassis_height/2 - 0.04}" rpy="0 0 0"/>
-  </joint>
-  <link name="frame_right">
-    <visual>
-      <geometry><box size="${chassis_length} 0.06 0.06"/></geometry>
-      <material name="chassis_steel"/>
-    </visual>
-    <inertial><mass value="0.01"/><inertia ixx="0.001" ixy="0" ixz="0" iyy="0.001" iyz="0" izz="0.001"/></inertial>
-  </link>
-  <!-- ═══════════════════════════════════════════
-       BODY PANELS
-       ═══════════════════════════════════════════ -->
-  <!-- Front nose panel -->
-  <joint name="front_panel_joint" type="fixed">
+  <gazebo reference="base_link"><material>Gazebo/White</material></gazebo>
+  <!-- SRM Blue accent stripes — flush with side faces -->
+  <joint name="stripe_l_jt" type="fixed">
+    <parent link="base_link"/><child link="stripe_l"/>
+    <origin xyz="0.10 ${cw/2 + 0.002} 0.06" rpy="0 0 0"/>
+  </joint>
+  <link name="stripe_l">
+    <visual><geometry><box size="${cl - 0.4} 0.005 0.08"/></geometry>
+      <material name="srm_blue"/></visual>
+    <xacro:tiny_inertial/>
+  </link>
+  <gazebo reference="stripe_l"><material>Gazebo/Blue</material></gazebo>
+  <joint name="stripe_r_jt" type="fixed">
+    <parent link="base_link"/><child link="stripe_r"/>
+    <origin xyz="0.10 ${-(cw/2 + 0.002)} 0.06" rpy="0 0 0"/>
+  </joint>
+  <link name="stripe_r">
+    <visual><geometry><box size="${cl - 0.4} 0.005 0.08"/></geometry>
+      <material name="srm_blue"/></visual>
+    <xacro:tiny_inertial/>
+  </link>
+  <gazebo reference="stripe_r"><material>Gazebo/Blue</material></gazebo>
+  <!-- Frame rails -->
+  <joint name="frame_l_jt" type="fixed">
+    <parent link="base_link"/><child link="frame_l"/>
+    <origin xyz="0 ${cw/2 - 0.08} ${-ch/2 - 0.03}" rpy="0 0 0"/>
+  </joint>
+  <link name="frame_l">
+    <visual><geometry><box size="${cl} 0.06 0.05"/></geometry>
+      <material name="dark_grey"/></visual>
+    <xacro:tiny_inertial/>
+  </link>
+  <joint name="frame_r_jt" type="fixed">
+    <parent link="base_link"/><child link="frame_r"/>
+    <origin xyz="0 ${-(cw/2 - 0.08)} ${-ch/2 - 0.03}" rpy="0 0 0"/>
+  </joint>
+  <link name="frame_r">
+    <visual><geometry><box size="${cl} 0.06 0.05"/></geometry>
+      <material name="dark_grey"/></visual>
+    <xacro:tiny_inertial/>
+  </link>
+  <!-- ── Body panels ── -->
+  <joint name="front_panel_jt" type="fixed">
     <parent link="base_link"/><child link="front_panel"/>
-    <origin xyz="${chassis_length/2 - 0.01} 0 0.10" rpy="0 0 0"/>
+    <origin xyz="${cl/2} 0 0.10" rpy="0 0 0"/>
   </joint>
   <link name="front_panel">
-    <visual>
-      <geometry><box size="0.10 ${chassis_width} 0.40"/></geometry>
-      <material name="arctic_white"/>
-    </visual>
-    <inertial><mass value="0.01"/><inertia ixx="0.001" ixy="0" ixz="0" iyy="0.001" iyz="0" izz="0.001"/></inertial>
-  </link>
+    <visual><geometry><box size="0.08 ${cw} 0.38"/></geometry>
+      <material name="white"/></visual>
+    <xacro:tiny_inertial/>
+  </link>
+  <gazebo reference="front_panel"><material>Gazebo/White</material></gazebo>
+  <!-- Front bumper (black) -->
+  <joint name="front_bump_jt" type="fixed">
+    <parent link="base_link"/><child link="front_bump"/>
+    <origin xyz="${cl/2 + 0.01} 0 ${-ch/2 + 0.05}" rpy="0 0 0"/>
+  </joint>
+  <link name="front_bump">
+    <visual><geometry><box size="0.10 ${cw + 0.06} 0.12"/></geometry>
+      <material name="chassis_blk"/></visual>
+    <xacro:tiny_inertial/>
+  </link>
+  <gazebo reference="front_bump"><material>Gazebo/DarkGrey</material></gazebo>
   <!-- Rear panel -->
-  <joint name="rear_panel_joint" type="fixed">
+  <joint name="rear_panel_jt" type="fixed">
     <parent link="base_link"/><child link="rear_panel"/>
-    <origin xyz="${-(chassis_length/2 - 0.01)} 0 0.10" rpy="0 0 0"/>
+    <origin xyz="${-cl/2} 0 0.10" rpy="0 0 0"/>
   </joint>
   <link name="rear_panel">
-    <visual>
-      <geometry><box size="0.10 ${chassis_width} 0.35"/></geometry>
-      <material name="arctic_white"/>
-    </visual>
-    <inertial><mass value="0.01"/><inertia ixx="0.001" ixy="0" ixz="0" iyy="0.001" iyz="0" izz="0.001"/></inertial>
-  </link>
-  <!-- Left side panel -->
-  <joint name="side_left_joint" type="fixed">
-    <parent link="base_link"/><child link="side_left"/>
-    <origin xyz="0.20 ${chassis_width/2} 0.15" rpy="0 0 0"/>
-  </joint>
-  <link name="side_left">
-    <visual>
-      <geometry><box size="${chassis_length - 0.5} 0.05 0.50"/></geometry>
-      <material name="arctic_white"/>
-    </visual>
-    <inertial><mass value="0.01"/><inertia ixx="0.001" ixy="0" ixz="0" iyy="0.001" iyz="0" izz="0.001"/></inertial>
-  </link>
-  <!-- Right side panel -->
-  <joint name="side_right_joint" type="fixed">
-    <parent link="base_link"/><child link="side_right"/>
-    <origin xyz="0.20 ${-chassis_width/2} 0.15" rpy="0 0 0"/>
-  </joint>
-  <link name="side_right">
-    <visual>
-      <geometry><box size="${chassis_length - 0.5} 0.05 0.50"/></geometry>
-      <material name="arctic_white"/>
-    </visual>
-    <inertial><mass value="0.01"/><inertia ixx="0.001" ixy="0" ixz="0" iyy="0.001" iyz="0" izz="0.001"/></inertial>
-  </link>
-  <!-- ═══════════════════════════════════════════
-       DASHBOARD
-       ═══════════════════════════════════════════ -->
-  <joint name="dashboard_joint" type="fixed">
-    <parent link="base_link"/><child link="dashboard"/>
-    <origin xyz="${chassis_length/2 - 0.55} 0 0.38" rpy="0 0.35 0"/>
-  </joint>
-  <link name="dashboard">
-    <visual>
-      <geometry><box size="0.08 ${chassis_width - 0.1} 0.35"/></geometry>
-      <material name="dashboard_blk"/>
-    </visual>
-    <inertial><mass value="0.01"/><inertia ixx="0.001" ixy="0" ixz="0" iyy="0.001" iyz="0" izz="0.001"/></inertial>
-  </link>
-  <!-- Steering column -->
-  <joint name="steering_col_joint" type="fixed">
-    <parent link="base_link"/><child link="steering_column"/>
-    <origin xyz="${chassis_length/2 - 0.50} 0.25 0.45" rpy="0 -0.6 0"/>
-  </joint>
-  <link name="steering_column">
-    <visual>
-      <geometry><cylinder radius="0.025" length="0.40"/></geometry>
-      <material name="dark_grey"/>
-    </visual>
-    <inertial><mass value="0.01"/><inertia ixx="0.001" ixy="0" ixz="0" iyy="0.001" iyz="0" izz="0.001"/></inertial>
-  </link>
-  <!-- Steering wheel -->
-  <joint name="steering_wheel_joint" type="fixed">
-    <parent link="steering_column"/><child link="steering_wheel"/>
-    <origin xyz="0 0 0.22" rpy="1.5708 0.5 0"/>
-  </joint>
-  <link name="steering_wheel">
-    <visual>
-      <geometry><cylinder radius="0.18" length="0.025"/></geometry>
-      <material name="dark_grey"/>
-    </visual>
-    <inertial><mass value="0.01"/><inertia ixx="0.001" ixy="0" ixz="0" iyy="0.001" iyz="0" izz="0.001"/></inertial>
-  </link>
-  <!-- ═══════════════════════════════════════════
-       WINDSHIELD
-       ═══════════════════════════════════════════ -->
-  <joint name="windshield_joint" type="fixed">
-    <parent link="base_link"/><child link="windshield"/>
-    <origin xyz="${chassis_length/2 - 0.42} 0 0.70" rpy="0 -0.30 0"/>
-  </joint>
-  <link name="windshield">
-    <visual>
-      <geometry><box size="${ws_thickness} ${chassis_width - 0.05} ${ws_height}"/></geometry>
-      <material name="clear_acrylic"/>
-    </visual>
-    <inertial><mass value="0.01"/><inertia ixx="0.001" ixy="0" ixz="0" iyy="0.001" iyz="0" izz="0.001"/></inertial>
-  </link>
-  <!-- ═══════════════════════════════════════════
-       ROOF PILLARS (A-front, B-rear)
-       ═══════════════════════════════════════════ -->
-  <!-- Front-left pillar -->
-  <joint name="pillar_fl_joint" type="fixed">
-    <parent link="base_link"/><child link="pillar_fl"/>
-    <origin xyz="${chassis_length/2 - 0.30} ${chassis_width/2 - 0.06} 0.75" rpy="0 0 0"/>
-  </joint>
-  <link name="pillar_fl">
-    <visual><geometry><cylinder radius="${pillar_r}" length="${pillar_h}"/></geometry><material name="arctic_white"/></visual>
-    <inertial><mass value="0.01"/><inertia ixx="0.001" ixy="0" ixz="0" iyy="0.001" iyz="0" izz="0.001"/></inertial>
-  </link>
-  <!-- Front-right pillar -->
-  <joint name="pillar_fr_joint" type="fixed">
-    <parent link="base_link"/><child link="pillar_fr"/>
-    <origin xyz="${chassis_length/2 - 0.30} ${-(chassis_width/2 - 0.06)} 0.75" rpy="0 0 0"/>
-  </joint>
-  <link name="pillar_fr">
-    <visual><geometry><cylinder radius="${pillar_r}" length="${pillar_h}"/></geometry><material name="arctic_white"/></visual>
-    <inertial><mass value="0.01"/><inertia ixx="0.001" ixy="0" ixz="0" iyy="0.001" iyz="0" izz="0.001"/></inertial>
-  </link>
-  <!-- Rear-left pillar -->
-  <joint name="pillar_rl_joint" type="fixed">
-    <parent link="base_link"/><child link="pillar_rl"/>
-    <origin xyz="${-(chassis_length/2 - 0.30)} ${chassis_width/2 - 0.06} 0.75" rpy="0 0 0"/>
-  </joint>
-  <link name="pillar_rl">
-    <visual><geometry><cylinder radius="${pillar_r}" length="${pillar_h}"/></geometry><material name="arctic_white"/></visual>
-    <inertial><mass value="0.01"/><inertia ixx="0.001" ixy="0" ixz="0" iyy="0.001" iyz="0" izz="0.001"/></inertial>
-  </link>
-  <!-- Rear-right pillar -->
-  <joint name="pillar_rr_joint" type="fixed">
-    <parent link="base_link"/><child link="pillar_rr"/>
-    <origin xyz="${-(chassis_length/2 - 0.30)} ${-(chassis_width/2 - 0.06)} 0.75" rpy="0 0 0"/>
-  </joint>
-  <link name="pillar_rr">
-    <visual><geometry><cylinder radius="${pillar_r}" length="${pillar_h}"/></geometry><material name="arctic_white"/></visual>
-    <inertial><mass value="0.01"/><inertia ixx="0.001" ixy="0" ixz="0" iyy="0.001" iyz="0" izz="0.001"/></inertial>
-  </link>
-  <!-- ═══════════════════════════════════════════
-       ROOF CANOPY (FRP)
-       ═══════════════════════════════════════════ -->
-  <joint name="roof_joint" type="fixed">
-    <parent link="base_link"/><child link="roof_link"/>
-    <origin xyz="-0.10 0 ${roof_height - chassis_z}" rpy="0 0 0"/>
-  </joint>
-  <link name="roof_link">
-    <visual>
-      <geometry><box size="${roof_length} ${roof_width + 0.10} ${roof_thickness}"/></geometry>
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
Commit message: fix: fixed the position of the buggy

File: src/buggy_description/urdf/buggy_urdf.xacro (robot description, xacro)
@@ -609,6 +609,6 @@
   <joint name="lidar_jt" type="fixed">
     <parent link="base_link"/><child link="lidar_link"/>
-    <!-- scan origin at 1.60m above base_link, offset -0.10 to align with roof -->
-    <origin xyz="-0.10 0.0 1.60" rpy="0 0 0"/>
+    <!-- scan origin at 1.85m above base_link, offset -0.10 to align with roof -->
+    <origin xyz="-0.10 0.0 1.85" rpy="0 0 0"/>
   </joint>
   <link name="lidar_link">

Commit message: feat: Team Charlie complete navigation stack — path planning, state machine, safety systems, full system launch

File: src/buggy_description/urdf/buggy_urdf.xacro (robot description, xacro)
@@ -91,5 +91,5 @@
       <mass value="280.0"/>
       <origin xyz="0 0 0" rpy="0 0 0"/>
-      <inertia ixx="80" ixy="0" ixz="0" iyy="400" iyz="0" izz="450"/>
+<inertia ixx="350" ixy="0" ixz="0" iyy="800" iyz="0" izz="900"/>
     </inertial>
   </link>
@@ -590,5 +590,5 @@
       </inertial>
     </link>
-<gazebo reference="${name}"><mu1>5.0</mu1><mu2>5.0</mu2><kp>1e7</kp><kd>1</kd><minDepth>0.001</minDepth><maxVel>0.1</maxVel><material>Gazebo/Black</material></gazebo>
+<gazebo reference="${name}"><mu1>1.0</mu1><mu2>1.0</mu2><kp>1e6</kp><kd>100</kd><minDepth>0.001</minDepth><maxVel>1.0</maxVel><material>Gazebo/Black</material></gazebo>
   </xacro:macro>
   <xacro:wheel name="wfl" px=" 1.30" py=" 0.55" side=" 1"/>
@@ -778,7 +778,7 @@
       <right_joint>wrr_jt</right_joint>
       <wheel_separation>1.10</wheel_separation>
-      <wheel_diameter>${wr * 2}</wheel_diameter>
-      <max_wheel_torque>500</max_wheel_torque>
-      <max_wheel_acceleration>5.0</max_wheel_acceleration>
+      <wheel_diameter>0.52</wheel_diameter>
+      <max_wheel_torque>200</max_wheel_torque>
+      <max_wheel_acceleration>1.0</max_wheel_acceleration>
       <publish_odom>true</publish_odom>
       <publish_odom_tf>true</publish_odom_tf>
@@ -788,4 +788,5 @@
       <command_topic>cmd_vel</command_topic>
       <odometry_topic>odom</odometry_topic>
+      <ros_debug_level>na</ros_debug_level>
     </plugin>
   </gazebo>
